File: fpga-banks-16-34.kicad_sch (KiCad schematic)
At the start: 24 parts, among them U3002 XC7K160T-FFG676, U9001 Oscillator_SMD_100MHz_ASFLMB, U9002 PCA9517A_TSSOP

Commit message: Start creating pinout and fanout for FPGA bank 33
Connections:
- net VREF_33 is gone; now on net VREF: C9004.1, C9005.1, R9013.2, R9014.1
- net ALERT_N: now also U3002.AD13 (IO_L17N_T2_33)
- net DQ12_A: now also U3002.AC18 (IO_L13P_T2_MRCC_32); no longer U3002.AD18 (IO_L13N_T2_MRCC_32)
- net DQ15_A: now also U3002.AD18 (IO_L13N_T2_MRCC_32); no longer U3002.AC18 (IO_L13P_T2_MRCC_32)
- net DQ2_B: now also U3002.AF3 (IO_L24P_T3_34); no longer U3002.AD3 (IO_L19N_T3_VREF_34)
- net DQ4_A: now also U3002.W15 (IO_L22P_T3_32); no longer U3002.W16 (IO_L22N_T3_32)
- net DQ5_A: now also U3002.W16 (IO_L22N_T3_32); no longer U3002.Y17 (IO_L19P_T3_32)
- net DQ6_A: now also U3002.Y17 (IO_L19P_T3_32); no longer U3002.W15 (IO_L22P_T3_32)
- net RESET_n: now also U3002.AF9 (IO_L24N_T3_33)
- net VRN: now also U3002.U9 (IO_0_VRN_33)
- net VRP: now also U3002.V12 (IO_25_VRP_33)
- net +1V1: now reaches U3002.AB18 (VCCO_32), U3002.AC15 (VCCO_32), U3002.AE19 (VCCO_32), U3002.AF16 (VCCO_32), U3002.W17 (VCCO_32), U3002.Y14 (VCCO_32)
- net +1V1: now also U3002.AA1 (VCCO_34), U3002.AA11 (VCCO_33), U3002.AB8 (VCCO_33), U3002.AC5 (VCCO_34), U3002.AD12 (VCCO_33), U3002.AD2 (VCCO_34), U3002.AE9 (VCCO_33), U3002.AF6 (VCCO_34), U3002.U3 (VCCO_34), U3002.V10 (VCCO_33), U3002.W7 (VCCO_33), U3002.Y4 (VCCO_34)
- net VREF: now reaches U3002.AE16 (IO_L6N_T0_VREF_32)
- net VREF: now also U3002.AD3 (IO_L19N_T3_VREF_34), U3002.AE11 (IO_L19N_T3_VREF_33), U3002.W4 (IO_L6N_T0_VREF_34), U3002.W8 (IO_L6N_T0_VREF_33), U3002.Y18 (IO_L19N_T3_VREF_32)
- net CK0_B_P: now reaches U3002.AA10 (IO_L14P_T2_SRCC_33)
- net CK0_B_N: now reaches U3002.AB10 (IO_L14N_T2_SRCC_33)
- net CK0_A_P: now reaches U3002.AB11 (IO_L13P_T2_MRCC_33)
- net CK0_A_N: now reaches U3002.AC11 (IO_L13N_T2_MRCC_33)
- net CK1_A_P: now reaches U3002.AE12 (IO_L21P_T3_DQS_33)
- net CK1_B_P: now reaches U3002.AE13 (IO_L23P_T3_33)
- net CK1_A_N: now reaches U3002.AF12 (IO_L21N_T3_DQS_33)
- net CK1_B_N: now reaches U3002.AF13 (IO_L23N_T3_33)
- no-connect marks 33 -> 41

Commit message: Finish pin assigment for bank 33
Connections:
- net CA0_A: now also U3002.AD11 (IO_L19P_T3_33)
- net CA0_B: now also U3002.V7 (IO_L2N_T0_33)
- net CA10_A: now also U3002.AC7 (IO_L10N_T1_33)
- net CA10_B: now also U3002.V11 (IO_L1P_T0_33)
- net CA11_A: now also U3002.AB7 (IO_L10P_T1_33)
- net CA11_B: now also U3002.W10 (IO_L3P_T0_DQS_33)
- net CA12_A: now also U3002.AA7 (IO_L8N_T1_33)
- net CA12_B: now also U3002.W11 (IO_L1N_T0_33)
- net CA1_A: now also U3002.AC12 (IO_L15N_T2_DQS_33)
- net CA1_B: now also U3002.Y7 (IO_L4N_T0_33)
- net CA2_A: now also U3002.AD10 (IO_L20P_T3_33)
- net CA2_B: now also U3002.V8 (IO_L2P_T0_33)
- net CA3_A: now also U3002.AC13 (IO_L17P_T2_33)
- net CA3_B: now also U3002.V9 (IO_L6P_T0_33)
- net CA4_A: now also U3002.AD9 (IO_L12N_T1_MRCC_33)
- net CA4_B: now also U3002.Y10 (IO_L5N_T0_33)
- net CA5_A: now also U3002.AC9 (IO_L12P_T1_MRCC_33)
- net CA5_B: now also U3002.Y11 (IO_L5P_T0_33)
- net CA6_A: now also U3002.AA9 (IO_L11P_T1_SRCC_33)
- net CA6_B: now also U3002.W9 (IO_L3N_T0_DQS_33)
- net CA7_A: now also U3002.AB9 (IO_L11N_T1_SRCC_33)
- net CA7_B: now also U3002.AA13 (IO_L16P_T2_33)
- net CA8_A: now also U3002.AC8 (IO_L9P_T1_DQS_33)
- net CA8_B: now also U3002.Y13 (IO_L18P_T2_33)
- net CA9_A: now also U3002.AA8 (IO_L8P_T1_33)
- net CA9_B: now also U3002.Y12 (IO_L18N_T2_33)
- net CS0_A_n: now also U3002.AA12 (IO_L16N_T2_33)
- net CS0_B_n: now also U3002.Y8 (IO_L4P_T0_33)
- net CS1_A_n: now also U3002.AB12 (IO_L15P_T2_DQS_33)
- net CS1_B_n: now also U3002.AF10 (IO_L24P_T3_33)
Other:
- note removed: "Mach names of this pin"

Commit message: Replace supply labels with proper symbols
Connections:
- net SCL_2V5 is gone; now on net HSCL: R9005.2, U9002.2 (SCL_{1})
- net SDA_2V5 is gone; now on net HSDA: R9004.2, U9002.3 (SDA_{1})
- net +1V1: now also R9013.1, R9015.2
- net VDDQ: no longer R9013.1, R9015.2
- net 3V3_SYS renamed +3V3
Other:
- note added: "TODO: Connect HSA to Serial adress select"
- note added: "TODO: low side 1V8? Remove event?"
- moved on the sheet: C9001, C9004, C9005, R9013, R9014
