File: supply.kicad_sch (KiCad schematic)
At the start: 141 parts, among them J3 BarrelJack_3167288, J8 PinHeader_1x3_P2.54mm_Drill1.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, Q11 BSS138PW, U18 MAX812REUS+T, U19 PAC1954T-E_VQFN, U20 PAC1954T-E_VQFN, U21 SN74AHCT1G125_SOT

Commit message: Rework ON/OFF controll WiP
Parts:
- removed C236: C_100n_0402, data-center-rdimm-ddr4-tester-footprints:C_0402_1005Metric, symbol data-center-rdimm-ddr4-tester:C_100n_0402
- removed R191: R_0R_0402, data-center-rdimm-ddr4-tester-footprints:R_0402_1005Metric, symbol data-center-rdimm-ddr4-tester:R_0R_0402
- removed R212: R_100k_0402, data-center-rdimm-ddr4-tester-footprints:R_0402_1005Metric, symbol data-center-rdimm-ddr4-tester:R_100k_0402
- removed R213: R_10k_0402, data-center-rdimm-ddr4-tester-footprints:R_0402_1005Metric, symbol data-center-rdimm-ddr4-tester:R_10k_0402
- removed U21: SN74AHCT1G125_SOT, data-center-rdimm-ddr4-tester-footprints:SOT-753, symbol data-center-rdimm-ddr4-tester:SN74AHCT1G125_SOT
Connections:
- net +3V3_AON: now also C232.1, C233.1, R192.1, U18.4 (VCC)
- net 5V0_SYS: no longer C232.1, C233.1, R192.1, U18.4 (VCC)
- net 12V_PCIe: no longer names the net of R?.1
- net SUP_MCU.PG_VCCINT: no longer names the net of U?.7 (PG)
- no-connect marks 3 -> 4
Other:
- moved on the sheet: C233

Commit message: Update designators and sync schematic with PCB
Parts:
- gave numbers to parts that had none: 96
- renumbered 0V6 to 0V10001, 1V0 to 1V10001, 1V8 to 1V10002, 1V2 to 1V10003, 2V5 to 2V10001, 3V3 to 3V10001, 5V0 to 5V10001, C232 to C10038, C233 to C10039, C234 to C10040, C235 to C10041, D11 to D10002, GND2 to GND10001, GND1 to GND10002, J3 to J10001, J8 to J10002, NT15 to NT10001, NT8 to NT10002, NT9 to NT10003, NT10 to NT10004, NT16 to NT10005, NT12 to NT10006, NT13 to NT10007, NT14 to NT10008, PHY1 to PHY10001, PWR1 to PWR10001, Q11 to Q10001, R124 to R10043, R192 to R10044, R194 to R10045, R195 to R10046, R119 to R10047, R162 to R10048, R202 to R10049, R203 to R10050, R204 to R10051, U18 to U10009, U19 to U10010, U20 to U10011, VIN1 to VIN10001

Commit message: Finish preliminary version of power supply sheet
Parts:
- removed 0V10001, 2V10001: TP_1mm_SMD, data-center-rdimm-ddr4-tester-footprints:Testpoint_smd_1mm, symbol data-center-rdimm-ddr4-tester:TP_1mm_SMD
- removed C10022: C_100n_0402, antmicro-footprints:C_0402_1005Metric, symbol antmicroCapacitors0402:C_100n_0402
- removed C10038: C_100n_0402, data-center-rdimm-ddr4-tester-footprints:C_0402_1005Metric, symbol data-center-rdimm-ddr4-tester:C_100n_0402
- removed D10001: BZX84C5V1-TP, antmicro-footprints:SOT-23-3, symbol antmicroDiodesZenerSingle:BZX84C5V1-TP
- removed D10002: PDS760, data-center-rdimm-ddr4-tester-footprints:PowerDI5, symbol data-center-rdimm-ddr4-tester:PDS760
- removed J10001: BarrelJack_3167288, data-center-rdimm-ddr4-tester-footprints:BarrelJack_3167288_Horizontal, symbol data-center-rdimm-ddr4-tester:BarrelJack_3167288
- removed NT10001, NT10002, NT10003, NT10004, NT10005, NT10006, NT10007, NT10008: Net-Tie_2, data-center-rdimm-ddr4-tester-footprints:NetTie-2_SMD_Pad0.127mm, symbol data-center-rdimm-ddr4-tester:Net-Tie_2
- removed PWR10001: LED_G_0603_KP-1608CGCK, data-center-rdimm-ddr4-tester-footprints:LED_0603_1608Metric_G, symbol data-center-rdimm-ddr4-tester:LED_G_0603_KP-1608CGCK
- removed R10001, R10002: R_47k_0402, antmicro-footprints:R_0402_1005Metric, symbol antmicroResistors0402:R_47k_0402
- removed R10004, R10005, R10006, R10007, R10008, R10009, R10010, R10011: R_0R_22.4A_0603, antmicro-footprints:R_0603_1608Metric, symbol antmicroResistors0603:R_0R_22.4A_0603
- removed R10012, R10023: R_0R_0402, antmicro-footprints:R_0402_1005Metric, symbol antmicroResistors0402:R_0R_0402
- removed R10047: R_330R_0402, data-center-rdimm-ddr4-tester-footprints:R_0402_1005Metric, symbol data-center-rdimm-ddr4-tester:R_330R_0402
- removed R10048, R10049, R10050, R10051: R_0R01_1206, data-center-rdimm-ddr4-tester-footprints:R_1206_3216Metric, symbol data-center-rdimm-ddr4-tester:R_0R01_1206
- removed U10005: SN74AHCT1G125_SOT, data-center-rdimm-ddr4-tester-footprints:SOT-753, symbol data-center-rdimm-ddr4-tester:SN74AHCT1G125_SOT
- added 1V2_MGTAVTT, 1V7, 1V8: TP_1mm_SMD, data-center-rdimm-ddr4-tester-footprints:Testpoint_smd_1mm, symbol data-center-rdimm-ddr4-tester:TP_1mm_SMD
- added C1001, C1002: C_100n_0402, antmicro-footprints:C_0402_1005Metric, symbol antmicroCapacitors0402:C_100n_0402
- added C1003: C_1u_25V_0603, antmicro-footprints:C_0603_1608Metric, symbol antmicroCapacitors0603:C_1u_25V_0603
- added D1001: ESDA25P35-1U1M, antmicro-footprints:ESDA25P35-1U1M, symbol antmicroTVSDiodes:ESDA25P35-1U1M
- added D1002: PMEG3050EP,115, antmicro-footprints:Nexperia_SOD128, symbol antmicroDiodesRectifiersSingle:PMEG3050EP,115
- added F1001: F_10A_1206, antmicro-footprints:F_1206_3216Metric, symbol antmicroFuses:F_10A_1206
- added J1001: BarrelJack_3167288, antmicro-footprints:BarrelJack_3167288_Horizontal, symbol antmicroBarrelAudioConnectors:BarrelJack_3167288
- added NT1001, NT1002, NT1003, NT1004, NT1005, NT1006, NT1007, NT1008, NT1009, NT1010, NT1011, NT1012, NT1013, NT1014: Net-Tie_2, data-center-rdimm-ddr4-tester-footprints:NetTie-2_SMD_Pad0.127mm, symbol data-center-rdimm-ddr4-tester:Net-Tie_2
- added Q1001: SI7613DN-T1-GE3, antmicro-footprints:Vishay_PowerPAK_1212-8_Single, symbol antmicroTransistorsFETsMOSFETsSingle:SI7613DN-T1-GE3
- added Q1002: BSS138PW, data-center-rdimm-ddr4-tester-footprints:SC70-3, symbol data-center-rdimm-ddr4-tester:BSS138PW
- added R1001: R_0R_22.4A_0603, antmicro-footprints:R_0603_1608Metric, symbol antmicroResistors0603:R_0R_22.4A_0603
- added R1002, R1003, R1004, R1005, R1006, R1007, R1008: R_0R01_1206, data-center-rdimm-ddr4-tester-footprints:R_1206_3216Metric, symbol data-center-rdimm-ddr4-tester:R_0R01_1206
- added SW1001: SW_CVS-02B, antmicro-footprints:SW_DIP_SPSTx02_Slide_Copal_CVS-02xB_W5.9mm_P1mm, symbol antmicroSlideSwitches:SW_CVS-02B
- added U1001: LTC4412IS6, antmicro-footprints:SOT-23-6, symbol antmicroPMICORControllersIdealDiodes:LTC4412IS6
- C10023: DNP DNP -> (none)
- renumbered 1V10002 to 1V0, 1V10001 to 1V0_MGTAVCC, 1V10003 to 1V1, PHY10001 to 1V2, 3V10001 to 3V3, 5V10001 to 5V0, VIN10001 to VDC
Connections:
- net 1V2_SYS is gone; now on net +1V2: 1V2.1
- net 5V0_SEN_+ is gone; now on net 3V3_SEN_+: U10011.11 (IN1+)
- net 5V0_SEN_- is gone; now on net 3V3_SEN_-: U10011.12 (IN1-)
- net VCC1V0 is gone; now on net +1V0_MGTAVCC: 1V0_MGTAVCC.1
- net VCC1V8 is gone; now on net +1V0: 1V0.1
- net VCC3V3 is gone; now on net +3V3: 3V3.1
- net VCC5V0 is gone; now on net +5V: 5V0.1
- net VDD1V2 is gone; now on net +1V1: 1V1.1
- net VIN is gone; now on net VDC: VDC.1
- net VPP_SEN_+ is gone; now on net 1V8_SEN_+: U10010.13 (IN2+)
- net VPP_SEN_- is gone; now on net 1V8_SEN_-: U10010.14 (IN2-)
- net +1V0_MGTAVCC: now also NT1008.2, R1002.2
- net +1V1: now also NT1014.2, R1008.2
- net +1V2: now also NT1010.2, R1004.2
- net +1V2_MGTAVTT: now also 1V2_MGTAVTT.1
- net +1V8: now also 1V8.1, NT1009.2, R1003.2
- net +3V3: now also C10040.1, C10041.1, R10045.1, R10046.1, U10010.2 (VDD), U10010.6 (ADDRSEL), U10011.2 (VDD), NT1012.2, R1006.2
- net +5V: now also NT1013.2, R1007.2
- net 1V1_local: now also NT1007.2, R1008.1
- net 1V2_local: now also NT1003.2, R1004.1
- net 1V7: now also 1V7.1, NT1011.2, R1005.2
- net 1V7_local: now also NT1004.2, R1005.1
- net 1V8_SEN_+: now also NT1002.1; no longer U10011.8 (IN3+)
- net 1V8_SEN_-: now also NT1009.1; no longer U10011.7 (IN3-)
- net 1V8_local: now also NT1002.2, R1003.1
- net 3V3_SEN_+: now also NT1005.1; no longer U10011.13 (IN2+)
- net 3V3_SEN_-: now also NT1012.1; no longer U10011.14 (IN2-)
- net 3V3_local: now also NT1005.2, R1001.2, R1006.1
- net 3V3_local_2: now also R1001.1
- net 5V_local: now also NT1006.2, R1007.1
- net GND: now also U10011.6 (ADDRSEL), C1001.1, C1002.1, C1003.1, D1001.1 (K), J1001.2, J1001.3, Q1002.2 (S), SW1001.SH, U1001.2 (GND), U1001.3 (CTL)
- net MGTAVCC_local: now also NT1001.2, R1002.1
- net PB_CTRL_OUT: now also SW1001.1
- net SEQ_EN: now also Q1002.3 (D), SW1001.4
- net VDC: now also C1003.2, D1002.1, Q1001.1 (S), Q1001.2 (S), Q1001.3 (S), U1001.6 (SENSE)
- net ~{PB_CTRL_CLR}: now reaches R10003.1, U10004.6 (~{CLR})
- net ~{PB_CTRL_CLR}: now also SW1001.3
- net 1V0_SEN_+ renamed 1V1_SEN_+
- net 1V1_SEN_+: now also NT1007.1
- net 1V0_SEN_- renamed 1V1_SEN_-
- net 1V1_SEN_-: now also NT1014.1
- removed net 3V3_SYS: C10040.1, C10041.1, R10045.1, R10046.1, U10010.2 (VDD), U10010.6 (ADDRSEL), U10011.2 (VDD), U10011.6 (ADDRSEL)
- net FPGA_PWR_DIS: no longer names the net of U10009.2 (~{RST})
- net FPGA_PWR_DIS: now also Q1002.1 (G)
- net PB_CTRL.~{PB_CTRL_INT} renamed ~{PB_CTRL_INT}
- net ~{PB_CTRL_INT}: now also SW1001.2
- net VCC1V2_SEN_+ renamed 1V7_SEN_+
- net 1V7_SEN_+: now also NT1004.1
- net VCC1V2_SEN_- renamed 1V7_SEN_-
- net 1V7_SEN_-: now also NT1011.1
- net VDDQ_SEN_+ renamed MGTAVCC_SEN_+
- net MGTAVCC_SEN_+: now also NT1001.1
- net VDDQ_SEN_- renamed MGTAVCC_SEN_-
- net MGTAVCC_SEN_-: now also NT1008.1
- net VTT_SEN_+ renamed 1V2_SEN_+
- net 1V2_SEN_+: now also NT1003.1
- net VTT_SEN_- renamed 1V2_SEN_-
- net 1V2_SEN_-: now also NT1010.1
- new net: C1001.2, C1002.2, D1001.2 (A), D1002.2, F1001.2, Q1001.5 (D), U1001.1 (IN)
- new net: F1001.1, J1001.1
- new net: Q1001.4 (G), U1001.5 (GATE)
- new net 5V_SEN_+: NT1006.1, U10011.8 (IN3+)
- new net 5V_SEN_-: NT1013.1, U10011.7 (IN3-)
- no-connect marks 4 -> 7
Other:
- note added: "DC JACK"
- note added: "FAN connector"
- note added: "I2C: 0x61"
- note added: "NOTE: 1. AUTO ON/ PB-Controller 2. 8s off/ instant off"
- note added: "Parallel output"
- note added: "Remove R302 and mount R295 after enabling parallel output"
- note removed: "DDR4"
- note removed: "Dual phase"
- note removed: "Input power connector"
- note removed: "Mount for instant shutdown"
- note removed: "NOTE2: when Res to GND mounted -> Alawys ON mount sequencer EN cap"
- note removed: "NOTE: mount 1/2"
- note removed: "NOTE: populate C339 and remove R308 when "Button controller" is not pupulated"
- note removed: "Optional FAN connector"
- note removed: "Remove R302 and mount R295 after enabling dual phase"
- note removed: "Shunt resistors Fuses"
- moved on the sheet: 1V0, 1V0_MGTAVCC, 1V1, 1V2, 3V3, 5V0, C10001, C10006, C10021, C10023, C10024, C10025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
