File: supply.kicad_sch (KiCad schematic)
At the start: 164 parts, among them J10001 JST_SH_1x4_BM04B-SRSS-TB-LF-SN, J1001 BarrelJack_3167288, Q10001 BSS138PW, Q10002 SI7613DN-T1-GE3, Q10003 BSS138PW, Q1001 SI7613DN-T1-GE3, Q1002 BSS138PW, Q20001 BSS138PW, SW10001 SW_DPDT_JS202011JCQN_SMD, SW1001 SW_CVS-02B, SW1002 SW_KMR211NGLFS_SMD, U10001 NCP718BSN330T1G, U10002 MPM54304GMN, U10003 MPM54304GMN, U10004 MAX16150A_SOT, U10005 LTC4412IS6, U10006 LM3880, U10007 MP8869S, U10008 XC6230H001ER-G, U10009 MAX812REUS+T, U1001 LTC4412IS6, U10010 PAC1954T-E_VQFN, U10011 PAC1954T-E_VQFN, U10012 MCP4726A0T-E_MAY

Commit message: Finish reworking power I2C and SPI termination
Parts:
- removed R10004, R10005, R10006, R10007: R_0R_0402, antmicro-footprints:R_0402_1005Metric, symbol antmicroResistors0402:R_0R_0402
- removed SW10001: SW_DPDT_JS202011JCQN_SMD, antmicro-footprints:SW_DPDT_CnK_JS202011JCQN_SMD, symbol antmicroSlideSwitches:SW_DPDT_JS202011JCQN_SMD
- removed SW1001: SW_CVS-02B, sodimm-ddr5-tester-footprints:SW_DIP_SPSTx02_Slide_Copal_CVS-02xB_W5.9mm_P1mm, symbol sodimm-ddr5-tester:SW_CVS-02B
- removed TP10003, TP10004, TP10006: TP_0.75mm_SMD, antmicro-footprints:TP_SMD_0.75mm, symbol antmicroTestPoints:TP_0.75mm_SMD
- added C10048, C10049: C_100n_0402, sodimm-ddr5-tester-footprints:C_0402_1005Metric, symbol sodimm-ddr5-tester:C_100n_0402
- added R10004, R10005: R_47k_0402, sodimm-ddr5-tester-footprints:R_0402_1005Metric, symbol sodimm-ddr5-tester:R_47k_0402
- added U10013, U10014: TS5A3359_VSSOP, antmicro-footprints:VSSOP-8_2.3x2mm_P0.5mm, symbol antmicroInterfaceAnalogSwitchesMultiplexersDemultiplexers:TS5A3359_VSSOP
- gave numbers to parts that had none: 1
Connections:
- net +3V3_AON: now also C10048.2, C10049.2, R10004.2, R10005.2, U10013.8 (VCC), U10014.8 (VCC)
- net FTDI_SCL_3V3: now also U10014.3 (NO3)
- net FTDI_SDA_3V3: now also U10013.3 (NO3)
- net GND: now also SW10002.13, SW10002.14, C10048.1, C10049.1, U10013.4 (GND), U10014.4 (GND)
- net PWR_SCL: now also U10002.4 (SCL), U10014.7 (COM); no longer U10010.4 (SCL), U10011.4 (SCL), U10012.2 (SCL)
- net PWR_SCL_3V3: now also U10014.2 (NO2)
- net PWR_SDA: now also SW10002.5, U10013.7 (COM); no longer U10010.5 (SDA), U10011.5 (SDA), U10012.3 (SDA)
- net PWR_SDA_3V3: now also U10013.2 (NO2)
- net SCL_3V3: now also U10014.1 (NO1)
- net SDA_3V3: now also U10013.1 (NO1)
- net PWR_SDA_2: now reaches SW10002.12
- net PWR_SDA_2: now also U10010.5 (SDA), U10011.5 (SDA), U10012.3 (SDA)
- net IN1: now reaches SW10002.3
- net IN1: now also R10004.1, U10013.6 (IN1), U10014.6 (IN1)
- net IN2: now reaches SW10002.4
- net IN2: now also R10005.1, U10013.5 (IN2), U10014.5 (IN2)
- net QDCDC1_SCL renamed PWR_SCL_2
- net PWR_SCL_2: now also U10010.4 (SCL), U10011.4 (SCL), U10012.2 (SCL); no longer U10002.4 (SCL)
Other:
- moved on the sheet: R10001, R10002, R10008, R10009, R10010, R10011

Commit message: SD card, flash, HDMI length matching and deskewing, add 0Ohm I2C mux bypass, Clean DRC, add DNP silkscreen marking, finish copper balancing
Parts:
- added R10006, R10007, R10024, R10044, R10047, R10048: R_0R_0402, sodimm-ddr5-tester-footprints:R_0402_1005Metric, symbol sodimm-ddr5-tester:R_0R_0402
Connections:
- net FTDI_SCL_3V3: now also R10048.2
- net FTDI_SDA_3V3: now also R10024.2
- net PWR_SCL: now also R10044.1, R10047.1, R10048.1
- net PWR_SCL_3V3: now also R10047.2
- net PWR_SDA: now also R10006.1, R10007.1, R10024.1
- net PWR_SDA_3V3: now also R10007.2
- net SCL_3V3: now also R10044.2
- net SDA_3V3: now also R10006.2
Other:
- moved on the sheet: C10043, C10044, C10045, C10046, C10047, C10048, C10049, R10001, R10002, R10004, R10005, R10008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
