File: fpga-bank-13-15.kicad_sch (KiCad schematic)
At the start: 3 parts, among them U4 XC7K160T-FFG676

Commit message: [#87036] Add IC testpoints
Other:
- company: (none) -> Antmicro Ltd.
Changed lines of the file:
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@@
 	(title_block
 		(title "SO-DIMM DDR5 Tester")
-		(date "2025-11-25")
+		(date "2025-11-26")
 		(rev "1.3.0")
+		(company "Antmicro Ltd.")
 		(comment 1 "www.antmicro.com")
 		(comment 2 "Antmicro Ltd")
