File: fpga-bank-16.kicad_sch (KiCad schematic)
At the start: 3 parts, among them U4 XC7K160T-FFG676, Y3 Oscillator_100MHz_ASFL1

Commit message: [#57478] ohp release
Parts:
- C164: footprint sodimm-ddr5-tester-footprints:C_0402_1005Metric -> antmicro-footprints:C_0402_1005Metric; symbol sodimm-ddr5-tester:C_100n_0402 -> antmicroCapacitors0402:C_100n_0402
- U4: footprint sodimm-ddr5-tester-footprints:BGA-676_27x27mm_Layout26x26_P1X1mm -> antmicro-footprints:BGA-676_27x27mm_Layout26x26_P1x1mm_FFG676; symbol sodimm-ddr5-tester:XC7K160T-FFG676 -> antmicroFPGAChips:XC7K160T-FFG676
- Y3: footprint sodimm-ddr5-tester-footprints:Oscillator_SMD_Abracon_ASFL1-4Pin_5.0x3.2mm -> antmicro-footprints:Oscillator_SMD_Abracon_ASFL1-4Pin_5.0x3.2mm; symbol sodimm-ddr5-tester:Oscillator_100MHz_ASFL1 -> antmicroOscillators:Oscillator_100MHz_ASFL1

Commit message: [#87036] Add IC testpoints
Other:
- company: (none) -> Antmicro Ltd.
Changed lines of the file:
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@@
 	(title_block
 		(title "SO-DIMM DDR5 Tester")
-		(date "2025-11-25")
+		(date "2025-11-26")
 		(rev "1.3.0")
+		(company "Antmicro Ltd.")
 		(comment 1 "www.antmicro.com")
 		(comment 2 "Antmicro Ltd")
