File: hyperram-flash.kicad_sch (KiCad schematic)
At the start: 17 parts, among them U1 IS66WVH16M8DBLL-100B1LI, U3 S25FL128SAGNFI000

Commit message: [#86301] Project refresh 81589
Parts:
- R10: DNP DNP -> (none)
